File: hardware/ricevitore/ricevitore.kicad_sch (KiCad schematic)
At the start: 0 parts

Commit message: Hardware: schema 0.1 del ricevitore USB
Chiavetta da collegare con lo stesso cavo al PC o al Raspberry Pi:
USB-C solo USB 2.0 (5,1 k su CC), USBLC6-2SC6 sulle linee dati,
AP2112K-3.3, CH340C alimentato a 3,3 V (V3 su VCC) per avere la UART ai
livelli del RAK3172, RAK3172 con IPEX su UART2. DTR e RTS non
collegati: pyserial li attiva aprendo la porta e il bridge non deve
resettare il modulo; pulsanti RESET e BOOT, pull-down su BOOT0, SWD per
il recupero. LED di alimentazione e LED su PA8 per i pacchetti ricevuti.

ERC di KiCad 10.0.7: una sola segnalazione, V3 del CH340C (uscita di
alimentazione nel simbolo) sulla rete di VOUT di U3, esclusa con la
motivazione nel .kicad_pro; netlist controllata rete per rete. README
di hardware aggiornato.

Co-Authored-By: Claude Opus 5.5 <noreply@anthropic.com>
Parts:
- added C1: 1µF, Capacitor_SMD:C_0805_2012Metric_Pad1.18x1.45mm_HandSolder, symbol Device:C
- added C2: 10µF, Capacitor_SMD:C_0805_2012Metric_Pad1.18x1.45mm_HandSolder, symbol Device:C
- added C3, C4, C5: 100nF, Capacitor_SMD:C_0805_2012Metric_Pad1.18x1.45mm_HandSolder, symbol Device:C
- added D1: verde, LED_SMD:LED_0805_2012Metric_Pad1.15x1.40mm_HandSolder, symbol Device:LED
- added D2: giallo, LED_SMD:LED_0805_2012Metric_Pad1.15x1.40mm_HandSolder, symbol Device:LED
- added J1: USB-C, Connector_USB:USB_C_Receptacle_HRO_TYPE-C-31-M-12, symbol Connector:USB_C_Receptacle_USB2.0_16P
- added J2: SWD, Connector_PinHeader_2.54mm:PinHeader_1x04_P2.54mm_Vertical, symbol Connector_Generic:Conn_01x04
- added R1, R2: 5.1k, Resistor_SMD:R_0805_2012Metric_Pad1.20x1.40mm_HandSolder, symbol Device:R
- added R3: 10k, Resistor_SMD:R_0805_2012Metric_Pad1.20x1.40mm_HandSolder, symbol Device:R
- added R4, R5: 1k, Resistor_SMD:R_0805_2012Metric_Pad1.20x1.40mm_HandSolder, symbol Device:R
- added SW1: RESET, Button_Switch_THT:SW_PUSH_6mm, symbol Switch:SW_Push
- added SW2: BOOT, Button_Switch_THT:SW_PUSH_6mm, symbol Switch:SW_Push
- added U1: RAK3172 EU868 con IPEX, RF_Module:RAK3172, symbol RF_Module:RAK3172-xx-8-SM-xI
- added U2: USBLC6-2SC6, Package_TO_SOT_SMD:SOT-23-6, symbol Power_Protection:USBLC6-2SC6
- added U3: AP2112K-3.3, Package_TO_SOT_SMD:SOT-23-5, symbol Regulator_Linear:AP2112K-3.3
- added U4: CH340C, Package_SO:SOIC-16_3.9x9.9mm_P1.27mm, symbol Interface_USB:CH340C
Connections:
- new net +3V3: C2.1, C3.1, C4.1, J2.1 (Pin_1), R4.1, SW2.2, U1.24 (VDD), U3.5 (VOUT), U4.16 (VCC), U4.4 (V3)
- new net BOOT0: R3.1, SW2.1, U1.21 (BOOT0)
- new net CC1: J1.A5 (CC1), R1.1
- new net CC2: J1.B5 (CC2), R2.1
- new net GND: C1.2, C2.2, C3.2, C4.2, C5.2, D1.1 (K), D2.1 (K), J1.A1 (GND), J1.A12 (GND), J1.B1 (GND), J1.B12 (GND), J1.SH (SHIELD), J2.4 (Pin_4), R1.2, R2.2, R3.2, SW1.2, U1.11 (GND), U1.17 (GND), U1.18 (GND), U1.23 (GND), U1.28 (GND), U2.2 (GND), U3.2 (GND), U4.1 (GND)
- new net LED_PWR_A: D1.2 (A), R4.2
- new net LED_RX: R5.1, U1.19 (PA8)
- new net LED_RX_A: D2.2 (A), R5.2
- new net NRST: C5.1, SW1.1, U1.22 (~{RST})
- new net SWCLK: J2.3 (Pin_3), U1.8 (PA14/SWCLK)
- new net SWDIO: J2.2 (Pin_2), U1.7 (PA13/SWDIO)
- new net UART2_RX: U1.1 (UART2_RX/PA3), U4.2 (TXD)
- new net UART2_TX: U1.2 (UART2_TX/PA2), U4.3 (RXD)
- new net USB_DM: J1.A7 (D-), J1.B7 (D-), U2.3 (I/O2), U2.4 (I/O2), U4.6 (UD-)
- new net USB_DP: J1.A6 (D+), J1.B6 (D+), U2.1 (I/O1), U2.6 (I/O1), U4.5 (UD+)
- new net VBUS: C1.1, J1.A4 (VBUS), J1.A9 (VBUS), J1.B4 (VBUS), J1.B9 (VBUS), U2.5 (VBUS), U3.1 (VIN), U3.3 (EN)
- no-connect marks 0 -> 31
Other:
- note added: "Ricevitore USB: si collega con lo stesso cavo al PC o al Raspberry Pi, che lo vedono come porta seriale (/dev/ttyUSB0, nome stabile in /dev/serial/by-id/). Alimentazione dalla USB, 5 V → 3,3 V con U3."
- note added: "U1: versione con connettore IPEX/u.FL, antenna esterna; pin RF non collegato. D2 su PA8: lampeggio a ogni pacchetto ricevuto, da aggiungere al firmware del ricevitore."
- note added: "U4 CH340C a 3,3 V: V3 collegato a VCC. DTR e RTS non collegati: il bridge (pyserial) li attiva aprendo la porta, e non deve resettare il modulo. Programmazione dalla stessa USB (Arduino, RUI3); se il bootloader non risponde: tenere BOOT, premere RESET, rilasciare; oppure SWD su J2."
